File: board/pico-opm-writer.kicad_sch (KiCad schematic)
At the start: 14 parts, among them J1 Conn_01x03, J2 Conn_01x03, J3 Conn_01x05, SW1 SW_Push, SW2 SW_Push, SW3 SW_Push, U1 YM2151

Commit message: 基板データの小修正
* YM2151のシンボルデータで12番ピンが非表示のピン情報で重複していたのを削除。
* C1の乗数記入漏れ
* 上記に合わせてPCBも更新(実質変更なし)
Parts:
- C1: value C_Small -> 0.1uF
Connections:
- net GND: no longer U1.12 (GND)
Changed lines of the file:
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@@
-		(pin "12"
-		)
 		(pin "12"
 		)
@@
 			)
 		)
-		(property "Value" "C_Small"
+		(property "Value" "0.1uF"
 			(at 247.65 34.2962 0)
 			(show_name no)
