File: board_pcba/pico-opm-writer_pcba.kicad_sch (KiCad schematic)
At the start: 72 parts, among them J1 USB-C 16P, J2 ST-005-G, J3 SWD, J4 UART, J5 DAC PROBE, SW1 SW_Push, SW2 SW_Push, SW3 SW_Push, SW4 SW_Push, U1 RP2350A, U2 W25Q128JVSIQ, U3 PCM5102A, U4 AMS1117-3.3, U5 XC6206P332MR, U6 YM2151, X1 12MHz

Commit message: RP2350A / PCM5102A 直載せ基板のレイアウトを起こす
board_pcba に回路図しか無かったところへ、配置・配線・GND ベタまで入れて
基板を一通り完成させる。46 × 47.5mm / 2 層 / 板厚 1.6mm。

配置は KiCad の pcbnew Python API で生成し、自動配線は Specctra DSN / SES 経由で
freerouting に投げた（DSN のエクスポートは GUI 専用で kicad-cli には無い）。
質が効くネット — 内蔵レギュレータのループ・USB 差動対・水晶・PCM5102A の
チャージポンプとアナログ出力 — だけは先に手で引いてロックしてある。

配線 753 本 / 総延長 1579mm（F.Cu 551 / B.Cu 202）。ビアは 167 本すべて
φ0.45mm / ドリル 0.2mm。アニュラーリングは 0.125mm で JLCPCB の推奨 0.13mm に
ほぼ一致し、同社自身の推奨ビア（φ0.35 / 0.2 → 0.075mm）より健全。ドリル 0.2mm は
能力表の推奨最小値で、0.3mm 未満なので基板製造費に小径穴の割増が付きうるが、
Economic PCBA（実装）の可否には影響しない。

配置と回転の意図は README §5.3 に書いた。U1 を 270 度回して GPIO2-11
(D0-D7 / A0 / /CS) の辺を真上の U6 へ向け、U6 を 90 度回して D2-D7 が U1 の
並び順のままソケットの上段へ抜けるようにしてある。U3 は 90 度回して I2S を上・
OUTL / OUTR を下に分け、PCM5102A のデータシート §12.1 の「I2S を出力から離す」を
パッケージの反対側に分けることで満たしている。

C8 / C10 のフットプリントを KiCad 標準の C_0402_1005Metric から、RPi の
リファレンス設計に入っていた専用 land pattern の複製 (rpi_capc1005x50_wide) へ
変更した。VREG_LX は U1 の 48 ピンから L1 まで、この 2 個のパッドの間を通る。
KiCad 標準はパッド間が 0.40mm しかなく 0.15mm 配線が物理的に通らない
（RPi の wide 品は 0.56mm）。これに気づかず標準品のままだと VREG_LX が
引けないので README §4.6 に理由を残した。出典と改変点は §6。

GND は F.Cu と B.Cu をまたぐ基板全面のゾーン 1 個に、5mm 格子のスティッチング
ビア 84 本。ゾーンは島の除去を「常に」にしてある。結果 F.Cu 7 領域（最大
1394mm²）/ B.Cu 3 領域（最大 1486mm²）で、すべての領域が 4 点以上で接続され、
1 点だけでぶら下がるアンテナ状のベタは無い。

回路図側の変更:

  J4 (UART) / J5 (DAC プローブ) / H3 / H4 を削除
  H1 / H2 を M3 から M2 (MountingHole_2.2mm_M2) へ
  未使用になった GP0 / GP1 に no-connect フラグ（TX / RX のラベルは撤去）
  C8 / C10 のフットプリントを差し替え

基板を詰めるためテストポイントは置いていない。Φ1 / SO / SH1 / SH2 を観測する
ときは U1 と U6 の間の配線にプローブを当てる（README §3.2）。

配線幅は Default 0.15 / Power・USB・VREG 0.2 / Analog 0.3mm。QFN-60 の
0.4mm ピッチの脱出部など 22 本だけ 0.125〜0.142mm にネックダウンしている。
JLCPCB の 1oz 標準能力は 0.10mm 幅 / 0.10mm 間隔なので製造上の問題はない。
min_track_width はこれに合わせて 0.12mm。

リファレンスのシルクは全て水平 (KeepUpright 有効) で 0.25mm グリッドに載せ、
68 個中 31 個が自分の部品から 0.5mm 以内、最も遠いもので 2.3mm。U1 の
デカップリング列と PCM5102A のアナログ部は 0402 が 1mm 間隔で並び、0.8mm の
文字が入る隙間が無いためここが限界。

C25 と R11 は DIP-24 ソケットの列間（15.24mm）に置いて面積を稼いでいる。
U6 のコートヤードの中に入るので、pico-opm-writer_p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
Parts:
- removed H3, H4: MountingHole, MountingHole:MountingHole_3.2mm_M3, symbol Mechanical:MountingHole
- removed J4: UART, Connector_PinHeader_2.54mm:PinHeader_1x03_P2.54mm_Vertical, symbol Connector_Generic:Conn_01x03
- removed J5: DAC PROBE, Connector_PinHeader_2.54mm:PinHeader_1x05_P2.54mm_Vertical, symbol Connector_Generic:Conn_01x05
- C10, C8: footprint Capacitor_SMD:C_0402_1005Metric -> pico-opm-writer:rpi_capc1005x50_wide
- H1, H2: footprint MountingHole:MountingHole_3.2mm_M3 -> MountingHole:MountingHole_2.2mm_M2
Connections:
- net RX: no longer names the net of U1.3 (GPIO1)
- net TX: no longer names the net of U1.2 (GPIO0)
- no-connect marks 7 -> 9
Other:
- note added: "GP0 / GP1 (UART) は未使用"
- note added: "H1 / H2 = M2 取付穴（対角 2 箇所）"
- note added: "J3 と U6・J2 は PCBA では実装しない（手はんだ）"
- note removed: "J3 / J4 / J5 と U6・J2 は PCBA では実装しない（手はんだ）"
